File: nanofrtpanel.sch (KiCad schematic (older format))
At the start: 10 parts, among them P1 CONN_02X08, Q1 BS170, SW1 DOWN, SW2 UP, SW3 SELECT, SW4 ESC, SW5 RESET

Commit message: Better access to RV1 and rebuild to be compatible.
Parts:
- removed SW5: RESET, Buttons_Switches_SMD:SW_SPST_PTS645, symbol SW_PUSH
- added JP1: Jumper_NO_Small, Pin_Headers:Pin_Header_Straight_1x02, symbol Jumper_NO_Small
- Q1: footprint Housings_TO-92:TO-92_Inline_Wide -> Housings_TO-92:TO-92_Inline_Narrow_Oval
Connections:
- net labels added: D11, D12, D2, D3, D4, D5, SW1, SW2, SW3, SW4, VDD, VSS
- net labels removed: D11a, D12a, D2a, D3a, D4a, D5a, RESETa, SW1a, SW2a, SW3a, SW4a, VDDa, VSSa
- wire segments 50 -> 54
- no-connect marks 6 -> 4
Other:
- note added: "Omit RV1 and Q1 if JP1 is closed.\nRV1 can be used here insted of main board."
Changed lines of the file:
@@
 EESchema Schematic File Version 2
+LIBS:nanofrtpanel-rescue
 LIBS:power
 LIBS:device
@@
 LIBS:contrib
 LIBS:valves
-LIBS:nanofrtpanel-cache
 EELAYER 25 0
 EELAYER END
@@
 Sheet 1 1
 Title "Arduino NANO TS-590S(G) front panel"
-Date "2015-07-19"
+Date "2015-07-21"
 Rev "1"
 Comp "by João Cunha lopes, CT2HME and Pedro Correia, CT7AEZ "
@@
 	4150 4600 4150 5700
 Text Label 4150 5650 1    60   ~ 0
-VDDa
+VDD
 Wire Wire Line
 	2750 4600 2750 5700
 Text Label 2750 5650 1    60   ~ 0
-VSSa
+VSS
 Wire Wire Line
 	2850 4600 2850 5700
 Text Label 2850 5650 1    60   ~ 0
-VDDa
+VDD
 $Comp
 L POT RV1
@@
 	5700 2450 6200 2450
 Text Label 6050 1850 0    60   ~ 0
-VDDa
+VDD
 Text Label 6050 2450 0    60   ~ 0
-VSSa
+VSS
 Text Label 6100 2150 0    60   ~ 0
 VO
@@
 	3050 4600 3050 5700
 Text Label 3050 5650 1    60   ~ 0
-D12a
+D12
 Wire Wire Line
 	3150 4600 3150 5700
 Text Label 3150 5650 1    60   ~ 0
-VSSa
+VSS
 Wire Wire Line
 	3250 4600 3250 5700
 Text Label 3250 5650 1    60   ~ 0
-D11a
+D11
 NoConn ~ 3350 4600
 NoConn ~ 3450 4600
@@
 	4050 4600 4050 5700
 Text Label 3750 5650 1    60   ~ 0
-D5a
+D5
 Text Label 3850 5650 1    60   ~ 0
-D4a
+D4
 Text Label 3950 5650 1    60   ~ 0
-D3a
+D3
 Text Label 4050 5650 1    60   ~ 0
-D2a
+D2
 Wire Wire Line
 	2600 1800 3350 1800
@@
 Wire Wire Line
 	2100 2100 1350 2100
-Text Label 3300 1800 2    60   ~ 0
-D12a
-Text Label 1400 1900 0    60   ~ 0
-D11a
-Text Label 3150 1900 0    60   ~ 0
-D5a
-Text Label 1400 2000 0    60   ~ 0
-D4a
-Text Label 3300 2000 2    60   ~ 0
-D3a
-Text Label 1400 2100 0    60   ~ 0
-D2a
+Text Label 3300 1900 2    60   ~ 0
+D12
+Text Label 3150 2000 0    60   ~ 0
+D11
+Text Label 1400 2300 0    60   ~ 0
+D5
+Text Label 3200 2300 0    60   ~ 0
+D4
+Text Label 1500 2400 2    60   ~ 0
+D3
+Text Label 3200 2400 0    60   ~ 0
+D2
 Wire Wire Line
 	2100 2200 1350 2200
@@
 L +5V #PWR01
 U 1 1 5514B6C8
-P 1750 1650
-F 0 "#PWR01" H 1750 1500 50  0001 C CNN
-F 1 "+5V" H 1750 1790 50  0000 C CNN
-F 2 "" H 1750 1650 60  0000 C CNN
-F 3 "" H 1750 1650 60  0000 C CNN
-	1    1750 1650
+P 2950 1500
+F 0 "#PWR01" H 2950 1350 50  0001 C CNN
+F 1 "+5V" H 2950 1640 50  0000 C CNN
+F 2 "" H 2950 1500 60  0000 C CNN
+F 3 "" H 2950 1500 60  0000 C CNN
+	1    2950 1500
 	-1   0    0    -1
 $EndComp
-Wire Wire Line
-	1750 1650 1750 1800
 $Comp
 L GND #PWR02
 U 1 1 5514B6D2
-P 3000 2600
-F 0 "#PWR02" H 3000 2350 50  0001 C CNN
-F 1 "GND" H 3000 2450 50  0000 C CNN
-F 2 "" H 3000 2600 60  0000 C CNN
-F 3 "" H 3000 2600 60  0000 C CNN
-	1    3000 2600
-	1    0    0    -1
+P 1750 1500
+F 0 "#PWR02" H 1750 1250 50  0001 C CNN
+F 1 "GND" H 1750 1350 50  0000 C CNN
+F 2 "" H 1750 1500 60  0000 C CNN
+F 3 "" H 1750 1500 60  0000 C CNN
+	1    1750 1500
+	-1   0    0    1
 $EndComp
 Wire Wire Line
 	2600 2200 3350 2200
-Text Label 3000 2200 0    60   ~ 0
-RESETa
-$Comp
-L SW_PUSH SW5
-U 1 1 5514D4D3
-P 9500 2850
-F 0 "SW5" H 9650 2960 50  0000 C CNN
-F 1 "RESET" H 9500 2770 50  0000 C CNN
-F 2 "Buttons_Switches_SMD:SW_SPST_PTS645" H 9500 2850 60  0001 C CNN
-F 3 "" H 9500 2850 60  0000 C CNN
-	1    9500 2850
-	1    0    0    -1
-$EndComp
 Wire Wire Line
 	2600 2400 3350 2400
 Wire Wire Line
 	2100 1800 1350 1800
-Text Label 1400 1800 0    60   ~ 0
-VDDa
-Text Label 3350 2400 2    60   ~ 0
-VSSa
+Text Label 3150 1800 0    60   ~ 0
+VDD
+Text Label 1550 1800 2    60   ~ 0
+VSS
 $Comp
 L C C1
@@
 	4950 2300 4950 2650
 Text Label 4950 1950 1    60   ~ 0
-VDDa
+VDD
 Text Label 4950 2600 1    60   ~ 0
-VSSa
+VSS
 $Comp
 L PWR_FLAG #FLG03
 U 1 1 5517E4F1
-P 1950 1550
-F 0 "#FLG03" H 1950 1645 50  0001 C CNN
-F 1 "PWR_FLAG" H 1950 1730 50  0000 C CNN
-F 2 "" H 1950 1550 60  0000 C CNN
-F 3 "" H 1950 1550 60  0000 C CNN
-	1    1950 1550
+P 2100 1500
+F 0 "#FLG03" H 2100 1595 50  0001 C CNN
+F 1 "PWR_FLAG" H 2100 1680 50  0000 C CNN
+F 2 "" H 2100 1500 60  0000 C CNN
+F 3 "" H 2100 1500 60  0000 C CNN
+	1    2100 1500
 	-1   0    0    -1
 $EndComp
@@
 L PWR_FLAG #FLG04
 U 1 1 5517E55A
-P 2750 2700
-F 0 "#FLG04" H 2750 2795 50  0001 C CNN
-F 1 "PWR_FLAG" H 2750 2880 50  0000 C CNN
-F 2 "" H 2750 2700 60  0000 C CNN
-F 3 "" H 2750 2700 60  0000 C CNN
-	1    2750 2700
-	-1   0    0    1
-$EndComp
-Wire Wire Line
-	1950 1550 1950 1800
-Connection ~ 1950 1800
+P 2600 1500
+F 0 "#FLG04" H 2600 1595 50  0001 C CNN
+F 1 "PWR_FLAG" H 2600 1680 50  0000 C CNN
+F 2 "" H 2600 1500 60  0000 C CNN
+F 3 "" H 2600 1500 60  0000 C CNN
+	1    2600 1500
+	1    0    0    -1
+$EndComp
 Wire Wire Line
 	9800 1650 9900 1650
-Wire Wire Line
-	9900 1650 9900 3300
-Text Label 9900 3250 1    60   ~ 0
-VSSa
 Wire Wire Line
 	9800 1950 9900 1950
 Connection ~ 9900 1950
 Wire Wire Line
-	9800 2250 9900 2250
+	9900 2250 9800 2250
 Connection ~ 9900 2250
 Wire Wire Line
-	9800 2550 9900 2550
+	9900 2550 9800 2550
 Connection ~ 9900 2550
 Wire Wire Line
-	9800 2850 9900 2850
-Connection ~ 9900 2850
-Wire Wire Line
 	9200 1650 8750 1650
 Wire Wire Line
@@
 Wire Wire Line
 	9200 2550 8750 2550
-Wire Wire Line
-	9200 2850 8750 2850
 Text Label 8800 1650 0    60   ~ 0
-SW1a
+SW1
 Text Label 8800 1950 0    60   ~ 0
-SW2a
+SW2
 Text Label 8800 2250 0    60   ~ 0
-SW3a
+SW3
 Text Label 8800 2550 0    60   ~ 0
-SW4a
-Text Label 8800 2850 0    60   ~ 0
-RESETa
+SW4
 Wire Wire Line
 	2600 2100 3350 2100
@@
 Wire Wire Line
 	2600 2300 3350 2300
-Text Label 3100 2100 0    60   ~ 0
-SW1a
-Text Label 1600 2200 2    60   ~ 0
-SW2a
-Text Label 1600 2300 2    60   ~ 0
-SW3a
-Text Label 3100 2300 0    60   ~ 0
-SW4a
-Wire Wire Line
-	2750 2700 2750 2400
-Connection ~ 2750 2400
-Wire Wire Line
-	3000 2600 3000 2400
-Connection ~ 1750 1800
-Connection ~ 3000 2400
+Text Label 1400 2100 0    60   ~ 0
+SW1
+Text Label 3300 2100 2    60   ~ 0
+SW2
+Text Label 1550 2200 2    60   ~ 0
+SW3
+Text Label 3150 2200 0    60   ~ 0
+SW4
 $Comp
 L CONN_02X08 P1
@@
 	1    0    0    -1
 $EndComp
-NoConn ~ 2100 2500
-NoConn ~ 2600 2500
 $Comp
 L BS170 Q1
@@
 F 0 "Q1" H 4350 6075 50  0000 L CNN
 F 1 "BS170" H 4350 6000 50  0000 L CNN
-F 2 "Housings_TO-92:TO-92_Inline_Wide" H 4350 5925 50  0000 L CIN
+F 2 "Housings_TO-92:TO-92_Inline_Narrow_Oval" H 4350 5925 50  0000 L CIN
 F 3 "" H 4150 6000 50  0000 L CNN
 	1    4150 6000
@@
 	4250 6200 4250 6750
 Text Label 4250 6700 1    60   ~ 0
-VSSa
+VSS
 Wire Wire Line
 	3950 6050 3400 6050
@@
 Wire Wire Line
 	1350 2400 2100 2400
-Text Label 1400 2400 0    60   ~ 0
+Text Label 3100 2500 0    60   ~ 0
 BCKL
+Wire Wire Line
+	1750 1500 1750 1800
+Connection ~ 1750 1800
+Wire Wire Line
+	2100 1500 2100 1800
+Wire Wire Line
+	2600 1500 2600 1800
+Wire Wire Line
+	2950 1500 2950 1800
+Connection ~ 2950 1800
+Wire Wire Line
+	2100 2500 1350 2500
+Wire Wire Line
+	2600 2500 3350 2500
+Text Label 1400 1900 0    60   ~ 0
+VO
+Text Label 1400 2000 0    60   ~ 0
+VSS
+Text Label 1400 2500 0    60   ~ 0
+VDD
+Wire Wire Line
+	9900 1650 9900 3050
+Text Label 9900 3000 1    60   ~ 0
+VSS
+$Comp
+L Jumper_NO_Small JP1
+U 1 1 55AE63BD
+P 4700 5800
+F 0 "JP1" H 4700 5880 50  0000 C CNN
+F 1 "Jumper_NO_Small" H 4710 5740 50  0001 C CNN
+F 2 "Pin_Headers:Pin_Header_Straight_1x02" H 4700 5800 60  0001 C CNN
+F 3 "" H 4700 5800 60  0000 C CNN
+	1    4700 5800
+	0    1    1    0
+$EndComp
+Wire Wire Line
+	4700 5900 4700 6300
+Wire Wire Line
+	4700 6300 4250 6300
+Connection ~ 4250 6300
+Wire Wire Line
+	4700 5700 4700 5600
+Wire Wire Line
+	4700 5600 4250 5600
+Connection ~ 4250 5600
+Text Notes 4550 5400 0    60   ~ 0
+Omit RV1 and Q1 if JP1 is closed.\nRV1 can be used here insted of main board.
 $EndSCHEMATC
